File: fpm_afe.kicad_sch (KiCad schematic)
At the start: 36 parts, among them J1 39301022, J2 132134, J3 132134, J4 878311420, U1 TPS7A4700xRGW, U2 PE43713B-Z, U3 ADL5536, U4 LFCN-800+, U5 LFCN-800+, U6 PAT-3+

Commit message: Finish schematic
Parts:
- removed C5: 0.1u, Capacitor_SMD:C_0603_1608Metric, symbol Device:C_Small
- removed U3: ADL5536, My_Footprints:RK_3_ADI, symbol My_Symbols:ADL5536
- removed U4, U5: LFCN-800+, My_Footprints:FV1206_MNC, symbol My_Symbols:LFCN-800+
- removed U6: PAT-3+, My_Footprints:Mini-Circuits_PAT-0plus_AF320_PL208, symbol My_Symbols:PAT-3+
- added C11: 0.1u, Capacitor_SMD:C_0603_1608Metric, symbol Device:C_Small
- added J5: 132134, My_Footprints:SMA_Amphenol_132134_Vertical, symbol My_Symbols:SMA-Straight-132134
- added U3: ADL5611, My_Footprints:RK_3_ADI, symbol My_Symbols:ADL5611
- added U4, U5: XLF-172H+, My_Footprints:QFN24_XLF-13H&plus__MNC, symbol My_Symbols:XLF-172H+
- added U7: RPS-2-30+, My_Footprints:TT1413_MNC, symbol My_Symbols:RPS-2-30+
- added U8: RCAT-01+, My_Footprints:RCAT_LZ1737, symbol My_Symbols:RCAT-01+
- L2: value 0603LS-471XJLC -> 43nH
Connections:
- net GND: now also J5.2 (Ext), U3.2 (G), U4.1 (NC), U4.10 (NC), U4.11 (NC), U4.12 (NC), U4.13 (NC), U4.14 (NC), U4.15 (GND), U4.17 (GND), U4.18 (NC), U4.19 (NC), U4.2 (GND), U4.20 (NC), U4.21 (NC), U4.22 (NC), U4.23 (NC), U4.24 (NC), U4.25 (PADDLE), U4.4 (GND), U4.5 (NC), U4.6 (NC), U4.7 (NC), U4.8 (NC), U4.9 (NC), U5.1 (NC), U5.10 (NC), U5.11 (NC), U5.12 (NC), U5.13 (NC), U5.14 (NC), U5.15 (GND), U5.17 (GND), U5.18 (NC), U5.19 (NC), U5.2 (GND), U5.20 (NC), U5.21 (NC), U5.22 (NC), U5.23 (NC), U5.24 (NC), U5.25 (PADDLE), U5.4 (GND), U5.5 (NC), U5.6 (NC), U5.7 (NC), U5.8 (NC), U5.9 (NC), U7.1 (GND), U7.2 (GND), U7.5 (GND), U8.2 (GND), U8.4 (GND)
- net at J2.1 (In): now also U8.1 (RF_IN)
- net at C6.2: now also U3.1
- net at C7.1, L2.2: now also U3.3
- net at C7.2: now also U5.3 (RF-IN)
- net at C8.1: now also U5.16 (RF-OUT)
- net at C4.1: now also U7.3 (PORT_2)
- new net: C11.1, U7.4 (PORT_1)
- new net: U4.16 (RF-OUT), U7.6 (SUM_PORT)
- new net: U4.3 (RF-IN), U8.3 (RF_OUT)
- new net: C11.2, J5.1 (In)
Other:
- note added: "Fill Pattern Monitor Front End"
- moved on the sheet: C1, C10, C12, C13, C14, C16, C17, C18, C2, C3, C4, C6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

Commit message: Board finished, gerbers generated
Parts:
- removed J2, J3, J5: 132134, My_Footprints:SMA_Amphenol_132134_Vertical, symbol My_Symbols:SMA-Straight-132134
- added J2, J3, J5: TMB-V5F2-3LC, My_Footprints:TMB-V5F2-3LC_PCBWay1_GCPW, symbol My_Symbols:SMA-TMB-V5F2-3LC
Connections:
- net GND: now also J2.2 (Ext), J3.2 (Ext), J5.2 (Ext)
- net at U8.1 (RF_IN): now also J2.1 (In)
- net at C8.2: now also J3.1 (In)
- net at C11.2: now also J5.1 (In)
Changed lines of the file:
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@@
 	)
 	(symbol
+		(lib_id "My_Symbols:SMA-TMB-V5F2-3LC")
+		(at 21.59 77.47 0)
+		(mirror y)
+		(unit 1)
+		(exclude_from_sim no)
+		(in_bom yes)
+		(on_board yes)
+		(dnp no)
+		(property "Reference" "J2"
+			(at 19.05 76.4931 0)
+			(effects
+				(font
+					(size 1.27 1.27)
+				)
+				(justify left)
+			)
+		)
+		(property "Value" "TMB-V5F2-3LC"
+			(at 29.972 72.898 0)
+			(effects
+				(font
+					(size 1.27 1.27)
+				)
+				(justify left)
+			)
+		)
+		(property "Footprint" "My_Footprints:TMB-V5F2-3LC_PCBWay1_GCPW"
+			(at 21.59 77.47 0)
+			(effects
+				(font
+					(size 1.27 1.27)
+				)
+				(hide yes)
+			)
+		)
+		(property "Datasheet" "~"
+			(at 21.59 77.47 0)
+			(effects
+				(font
+					(size 1.27 1.27)
+				)
+				(hide yes)
+			)
+		)
+		(property "Description" "coaxial connector (BNC, SMA, SMB, SMC, Cinch/RCA, LEMO, ...)"
+			(at 21.59 77.47 0)
+			(effects
+				(font
+					(size 1.27 1.27)
+				)
+				(hide yes)
+			)
+		)
+		(pin "1"
+		)
+		(pin "2"
+		)
+		(instances
+			(project "fpm_afe"
+				(path "/87d67133-f485-4ab6-855f-1bc7a1c63eff"
+					(reference "J2")
+					(unit 1)
+				)
+			)
+		)
+	)
+	(symbol
 		(lib_id "My_Symbols:+5.0V")
 		(at 232.41 93.98 0)
@@
 	)
 	(symbol
+		(lib_id "My_Symbols:SMA-TMB-V5F2-3LC")
+		(at 361.95 43.18 0)
+		(unit 1)
+		(exclude_from_sim no)
+		(in_bom yes)
+		(on_board yes)
+		(dnp no)
+		(property "Reference" "J5"
+			(at 364.49 42.2031 0)
+			(effects
+				(font
+					(size 1.27 1.27)
+				)
+				(justify left)
+			)
+		)
+		(property "Value" "TMB-V5F2-3LC"
+			(at 355.854 38.608 0)
+			(effects
+				(font
+					(size 1.27 1.27)
+				)
+				(justify left)
+			)
+		)
+		(property "Footprint" "My_Footprints:TMB-V5F2-3LC_PCBWay1_GCPW"
+			(at 361.95 43.18 0)
+			(effects
+				(font
+					(size 1.27 1.27)
+				)
+				(hide yes)
+			)
+		)
+		(property "Datasheet" "~"
+			(at 361.95 43.18 0)
+			(effects
+				(font
+					(size 1.27 1.27)
+				)
+				(hide yes)
+			)
+		)
+		(property "Description" "coaxial connector (BNC, SMA, SMB, SMC, Cinch/RCA, LEMO, ...)"
+			(at 361.95 43.18 0)
+			(effects
+				(font
+					(size 1.27 1.27)
+				)
+				(hide yes)
+			)
+		)
+		(pin "1"
+		)
+		(pin "2"
+		)
+		(instances
+			(project "fpm_afe"
+				(path "/87d67133-f485-4ab6-855f-1bc7a1c63eff"
+					(reference "J5")
+					(unit 1)
+				)
+			)
+		)
+	)
+	(symbol
 		(lib_id "My_Symbols:RCAT-01+")
 		(at 34.29 78.74 0)
@@
 	)
 	(symbol
-		(lib_id "My_Symbols:SMA-Straight-132134")
-		(at 21.59 77.47 0)
-		(mirror y)
-		(unit 1)
-		(exclude_from_sim no)
-		(in_bom yes)
-		(on_board yes)
-		(dnp no)
-		(property "Reference" "J2"
-			(at 24.892 80.518 0)
-			(effects
-				(font
-					(size 1.27 1.27)
-				)
-				(justify left)
-			)
-		)
-		(property "Value" "132134"
-			(at 24.892 73.152 0)
-			(effects
-				(font
-					(size 1.27 1.27)
-				)
-				(justify left)
-			)
-		)
-		(property "Footprint" "My_Footprints:SMA_Amphenol_132134_Vertical"
-			(at 21.59 77.47 0)
-			(effects
-				(font
-					(size 1.27 1.27)
-				)
-				(hide yes)
-			)
-		)
-		(property "Datasheet" "~"
-			(at 21.59 77.47 0)
-			(effects
-				(font
-					(size 1.27 1.27)
-				)
-				(hide yes)
-			)
-		)
-		(property "Description" "coaxial connector (BNC, SMA, SMB, SMC, Cinch/RCA, LEMO, ...)"
-			(at 21.59 77.47 0)
-			(effects
-				(font
-					(size 1.27 1.27)
-				)
-				(hide yes)
-			)
-		)
-		(pin "1"
-		)
-		(pin "2"
-		)
-		(instances
-			(project "fpm_afe"
-				(path "/87d67133-f485-4ab6-855f-1bc7a1c63eff"
-					(reference "J2")
-					(unit 1)
-				)
-			)
-		)
-	)
-	(symbol
 		(lib_id "power:GND")
 		(at 134.62 228.6 0)
@@
 	)
 	(symbol
-		(lib_id "My_Symbols:SMA-Straight-132134")
-		(at 386.08 137.16 0)
-		(unit 1)
-		(exclude_from_sim no)
-		(in_bom yes)
-		(on_board yes)
-		(dnp no)
-		(fields_autoplaced yes)
-		(property "Reference" "J3"
-			(at 388.62 136.1831 0)
-			(effects
-				(font
-					(size 1.27 1.27)
-				)
-				(justify left)
-			)
-		)
-		(property "Value" "132134"
-			(at 388.62 138.7231 0)
-			(effects
-				(font
-					(size 1.27 1.27)
-				)
-				(justify left)
-			)
-		)
-		(property "Footprint" "My_Footprints:SMA_Amphenol_132134_Vertical"
-			(at 386.08 137.16 0)
-			(effects
-				(font
-					(size 1.27 1.27)
-				)
-				(hide yes)
-			)
-		)
-		(property "Datasheet" "~"
-			(at 386.08 137.16 0)
-			(effects
-				(font
-					(size 1.27 1.27)
-				)
-				(hide yes)
-			)
-		)
-		(property "Description" "coaxial connector (BNC, SMA, SMB, SMC, Cinch/RCA, LEMO, ...)"
-			(at 386.08 137.16 0)
-			(effects
-				(font
-					(size 1.27 1.27)
-				)
-				(hide yes)
-			)
-		)
-		(pin "2"
-		)
-		(pin "1"
-		)
-		(instances
-			(project "fpm_afe"
-				(path "/87d67133-f485-4ab6-855f-1bc7a1c63eff"
-					(reference "J3")
-					(unit 1)
-				)
-			)
-		)
-	)
-	(symbol
 		(lib_id "power:GND")
 		(at 303.53 82.55 0)
@@
 	)
 	(symbol
+		(lib_id "My_Symbols:SMA-TMB-V5F2-3LC")
+		(at 386.08 137.16 0)
+		(unit 1)
+		(exclude_from_sim no)
+		(in_bom yes)
+		(on_board yes)
+		(dnp no)
+		(property "Reference" "J3"
+			(at 388.62 136.1831 0)
+			(effects
+				(font
+					(size 1.27 1.27)
+				)
+				(justify left)
+			)
+		)
+		(property "Value" "TMB-V5F2-3LC"
+			(at 379.984 132.842 0)
+			(effects
+				(font
+					(size 1.27 1.27)
+				)
+				(justify left)
+			)
+		)
+		(property "Footprint" "My_Footprints:TMB-V5F2-3LC_PCBWay1_GCPW"
+			(at 386.08 137.16 0)
+			(effects
+				(font
+					(size 1.27 1.27)
+				)
+				(hide yes)
+			)
+		)
+		(property "Datasheet" "~"
+			(at 386.08 137.16 0)
+			(effects
+				(font
+					(size 1.27 1.27)
+				)
+				(hide yes)
+			)
+		)
+		(property "Description" "coaxial connector (BNC, SMA, SMB, SMC, Cinch/RCA, LEMO, ...)"
+			(at 386.08 137.16 0)
+			(effects
+				(font
+					(size 1.27 1.27)
+				)
+				(hide yes)
+			)
+		)
+		(pin "1"
+		)
+		(pin "2"
+		)
+		(instances
+			(project "fpm_afe"
+				(path "/87d67133-f485-4ab6-855f-1bc7a1c63eff"
+					(reference "J3")
+					(unit 1)
+				)
+			)
+		)
+	)
+	(symbol
 		(lib_id "Device:C_Small")
 		(at 297.18 80.01 90)
@@
 					(unit 1)
 				)
-			)
-		)
-	)
-	(symbol
-		(lib_id "My_Symbols:SMA-Straight-132134")
-		(at 361.95 43.18 0)
-		(unit 1)
-		(exclude_from_sim no)
-		(in_bom yes)
-		(on_board yes)
-		(dnp no)
-		(fields_autoplaced yes)
-		(property "Reference" "J5"
-			(at 364.49 42.2031 0)
-			(effects
-				(font
-					(size 1.27 1.27)
-				)
-				(justify left)
-			)
-		)
-		(property "Value" "132134"
-			(at 364.49 44.7431 0)
-			(effects
-				(font
-					(size 1.27 1.27)
-				)
-				(justify left)
-			)
-		)
-		(property "Footprint" "My_Footprints:SMA_Amphenol_132134_Vertical"
-			(at 361.95 43.18 0)
-			(effects
-				(font
-					(size 1.27 1.27)
-				)
-				(hide yes)
-			)
-		)
-		(property "Datasheet" "~"
-			(at 361.95 43.18 0)
-			(effects
-				(font
-					(size 1.27 1.27)
-				)
-				(hide yes)
-			)
-		)
-		(property "Description" "coaxial connector (BNC, SMA, SMB, SMC, Cinch/RCA, LEMO, ...)"
-			(at 361.95 43.18 0)
-			(effects
-				(font
-					(size 1.27 1.27)
-				)
-				(hide yes)
-			)
-		)
-		(pin "2"
-		)
-		(pin "1"
-		)
-		(instances
-			(project "fpm_afe"
-				(path "/87d67133-f485-4ab6-855f-1bc7a1c63eff"
-					(reference "J5")
-					(unit 1)
-				)
